File: Hardware/BMU/BMU-CAN.kicad_sch (KiCad schematic)
At the start: 6 parts, among them U5 MCP2562FDT-H_SN

Commit message: update power part
Parts:
- renumbered C17 to C16, C16 to C17, CR1 to CR2, R14 to R23, R16 to R24, U5 to U6
Changed lines of the file:
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@@
 		(dnp no)
 		(fields_autoplaced yes)
-		(property "Reference" "#PWR08"
+		(property "Reference" "#PWR031"
 			(at 208.28 166.37 0)
 			(hide yes)
@@
 			(project "BMU"
 				(path "/efb70416-ce55-4766-98ba-c3d23efcccb1/ebb995bd-0019-4c04-a0dd-2962c6aaae17"
-					(reference "#PWR08")
+					(reference "#PWR031")
 					(unit 1)
 				)
@@
 		(in_pos_files yes)
 		(dnp no)
-		(property "Reference" "R16"
+		(property "Reference" "R24"
 			(at 226.06 137.16 0)
 			(show_name no)
@@
 			(project "BMU"
 				(path "/efb70416-ce55-4766-98ba-c3d23efcccb1/ebb995bd-0019-4c04-a0dd-2962c6aaae17"
-					(reference "R16")
+					(reference "R24")
 					(unit 1)
 				)
@@
 		(dnp no)
 		(fields_autoplaced yes)
-		(property "Reference" "C17"
+		(property "Reference" "C16"
 			(at 207.0163 110.49 90)
 			(show_name no)
@@
 			(project "BMU"
 				(path "/efb70416-ce55-4766-98ba-c3d23efcccb1/ebb995bd-0019-4c04-a0dd-2962c6aaae17"
-					(reference "C17")
+					(reference "C16")
 					(unit 1)
 				)
@@
 		(in_pos_files yes)
 		(dnp no)
-		(property "Reference" "R14"
+		(property "Reference" "R23"
 			(at 192.024 142.748 0)
 			(show_name no)
@@
 			(project "BMU"
 				(path "/efb70416-ce55-4766-98ba-c3d23efcccb1/ebb995bd-0019-4c04-a0dd-2962c6aaae17"
-					(reference "R14")
+					(reference "R23")
 					(unit 1)
 				)
@@
 		(in_pos_files yes)
 		(dnp no)
-		(property "Reference" "U5"
+		(property "Reference" "U6"
 			(at 209.042 123.444 0)
 			(show_name no)
@@
 			(project "BMU"
 				(path "/efb70416-ce55-4766-98ba-c3d23efcccb1/ebb995bd-0019-4c04-a0dd-2962c6aaae17"
-					(reference "U5")
+					(reference "U6")
 					(unit 1)
 				)
@@
 		(dnp no)
 		(fields_autoplaced yes)
-		(property "Reference" "#PWR028"
+		(property "Reference" "#PWR035"
 			(at 281.94 161.29 0)
 			(hide yes)
@@
 			(project "BMU"
 				(path "/efb70416-ce55-4766-98ba-c3d23efcccb1/ebb995bd-0019-4c04-a0dd-2962c6aaae17"
-					(reference "#PWR028")
+					(reference "#PWR035")
 					(unit 1)
 				)
@@
 		(dnp no)
 		(fields_autoplaced yes)
-		(property "Reference" "#PWR011"
+		(property "Reference" "#PWR033"
 			(at 222.25 116.84 0)
 			(hide yes)
@@
 			(project "BMU"
 				(path "/efb70416-ce55-4766-98ba-c3d23efcccb1/ebb995bd-0019-4c04-a0dd-2962c6aaae17"
-					(reference "#PWR011")
+					(reference "#PWR033")
 					(unit 1)
 				)
@@
 		(dnp no)
 		(fields_autoplaced yes)
-		(property "Reference" "CR1"
+		(property "Reference" "CR2"
 			(at 262.89 144.78 0)
 			(show_name no)
@@
 			(project "BMU"
 				(path "/efb70416-ce55-4766-98ba-c3d23efcccb1/ebb995bd-0019-4c04-a0dd-2962c6aaae17"
-					(reference "CR1")
+					(reference "CR2")
 					(unit 1)
 				)
@@
 		(dnp no)
 		(fields_autoplaced yes)
-		(property "Reference" "#PWR09"
+		(property "Reference" "#PWR032"
 			(at 214.63 116.84 0)
 			(hide yes)
@@
 			(project "BMU"
 				(path "/efb70416-ce55-4766-98ba-c3d23efcccb1/ebb995bd-0019-4c04-a0dd-2962c6aaae17"
-					(reference "#PWR09")
+					(reference "#PWR032")
 					(unit 1)
 				)
@@
 		(dnp no)
 		(fields_autoplaced yes)
-		(property "Reference" "#PWR014"
+		(property "Reference" "#PWR034"
 			(at 234.95 125.73 0)
 			(hide yes)
@@
 			(project "BMU"
 				(path "/efb70416-ce55-4766-98ba-c3d23efcccb1/ebb995bd-0019-4c04-a0dd-2962c6aaae17"
-					(reference "#PWR014")
+					(reference "#PWR034")
 					(unit 1)
 				)
@@
 		(in_pos_files yes)
 		(dnp no)
-		(property "Reference" "#PWR025"
+		(property "Reference" "#PWR030"
 			(at 201.93 124.46 0)
 			(hide yes)
@@
 			(project "BMU"
 				(path "/efb70416-ce55-4766-98ba-c3d23efcccb1/ebb995bd-0019-4c04-a0dd-2962c6aaae17"
-					(reference "#PWR025")
+					(reference "#PWR030")
 					(unit 1)
 				)
@@
 		(dnp no)
 		(fields_autoplaced yes)
-		(property "Reference" "C16"
+		(property "Reference" "C17"
 			(at 229.8763 110.49 90)
 			(show_name no)
@@
 			(project "BMU"
 				(path "/efb70416-ce55-4766-98ba-c3d23efcccb1/ebb995bd-0019-4c04-a0dd-2962c6aaae17"
-					(reference "C16")
-					(unit 1)
-				)
+					(reference "C17")
+					(unit 1)
+				)

Commit message: finish BMU, add test point + comment
Parts:
- added TP17, TP18: TestPoint_Small, TestPoint:TestPoint_THTPad_D1.5mm_Drill0.7mm, symbol Connector:TestPoint_Small
- R27: renamed from R24; now not fitted
- renumbered R23 to R26
Connections:
- net CANH: now also TP18.1
- net CANL: now also TP17.1
Changed lines of the file:
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@@
+	)
+	(junction
+		(at 264.16 135.89)
+		(diameter 0)
+		(color 0 0 0 0)
+	)
+	(junction
+		(at 264.16 140.97)
+		(diameter 0)
+		(color 0 0 0 0)
 	)
 	(junction
@@
 		(dnp no)
 		(fields_autoplaced yes)
-		(property "Reference" "#PWR031"
+		(property "Reference" "#PWR034"
 			(at 208.28 166.37 0)
 			(hide yes)
@@
 			(project "BMU"
 				(path "/efb70416-ce55-4766-98ba-c3d23efcccb1/ebb995bd-0019-4c04-a0dd-2962c6aaae17"
-					(reference "#PWR031")
+					(reference "#PWR034")
 					(unit 1)
 				)
@@
 		(on_board yes)
 		(in_pos_files yes)
-		(dnp no)
-		(property "Reference" "R24"
+		(dnp yes)
+		(property "Reference" "R27"
 			(at 226.06 137.16 0)
 			(show_name no)
@@
 			(project "BMU"
 				(path "/efb70416-ce55-4766-98ba-c3d23efcccb1/ebb995bd-0019-4c04-a0dd-2962c6aaae17"
-					(reference "R24")
+					(reference "R27")
 					(unit 1)
 				)
@@
 		(in_pos_files yes)
 		(dnp no)
-		(property "Reference" "R23"
+		(property "Reference" "R26"
 			(at 192.024 142.748 0)
 			(show_name no)
@@
 			(project "BMU"
 				(path "/efb70416-ce55-4766-98ba-c3d23efcccb1/ebb995bd-0019-4c04-a0dd-2962c6aaae17"
-					(reference "R23")
+					(reference "R26")
 					(unit 1)
 				)
@@
 		(dnp no)
 		(fields_autoplaced yes)
-		(property "Reference" "#PWR035"
+		(property "Reference" "#PWR038"
 			(at 281.94 161.29 0)
 			(hide yes)
@@
 			(project "BMU"
 				(path "/efb70416-ce55-4766-98ba-c3d23efcccb1/ebb995bd-0019-4c04-a0dd-2962c6aaae17"
-					(reference "#PWR035")
+					(reference "#PWR038")
+					(unit 1)
+				)
+			)
+		)
+	)
+	(symbol
+		(lib_id "Connector:TestPoint_Small")
+		(at 264.16 135.89 0)
+		(unit 1)
+		(body_style 1)
+		(exclude_from_sim no)
+		(in_bom yes)
+		(on_board yes)
+		(in_pos_files yes)
+		(dnp no)
+		(fields_autoplaced yes)
+		(property "Reference" "TP17"
+			(at 265.43 134.6199 0)
+			(show_name no)
+			(do_not_autoplace no)
+			(effects
+				(font
+					(size 1.27 1.27)
+				)
+				(justify left)
+			)
+		)
+		(property "Value" "TestPoint_Small"
+			(at 265.43 137.1599 0)
+			(hide yes)
+			(show_name no)
+			(do_not_autoplace no)
+			(effects
+				(font
+					(size 1.27 1.27)
+				)
+				(justify left)
+			)
+		)
+		(property "Footprint" "TestPoint:TestPoint_THTPad_D1.5mm_Drill0.7mm"
+			(at 269.24 135.89 0)
+			(hide yes)
+			(show_name no)
+			(do_not_autoplace no)
+			(effects
+				(font
+					(size 1.27 1.27)
+				)
+			)
+		)
+		(property "Datasheet" ""
+			(at 269.24 135.89 0)
+			(hide yes)
+			(show_name no)
+			(do_not_autoplace no)
+			(effects
+				(font
+					(size 1.27 1.27)
+				)
+			)
+		)
+		(property "Description" "test point"
+			(at 264.16 135.89 0)
+			(hide yes)
+			(show_name no)
+			(do_not_autoplace no)
+			(effects
+				(font
+					(size 1.27 1.27)
+				)
+			)
+		)
+		(pin "1"
+		)
+		(instances
+			(project "BMU"
+				(path "/efb70416-ce55-4766-98ba-c3d23efcccb1/ebb995bd-0019-4c04-a0dd-2962c6aaae17"
+					(reference "TP17")
 					(unit 1)
 				)
@@
 		(dnp no)
 		(fields_autoplaced yes)
-		(property "Reference" "#PWR033"
+		(property "Reference" "#PWR036"
 			(at 222.25 116.84 0)
 			(hide yes)
@@
 			(project "BMU"
 				(path "/efb70416-ce55-4766-98ba-c3d23efcccb1/ebb995bd-0019-4c04-a0dd-2962c6aaae17"
-					(reference "#PWR033")
+					(reference "#PWR036")
 					(unit 1)
 				)
@@
 		(dnp no)
 		(fields_autoplaced yes)
-		(property "Reference" "#PWR032"
+		(property "Reference" "#PWR035"
 			(at 214.63 116.84 0)
 			(hide yes)
@@
 			(project "BMU"
 				(path "/efb70416-ce55-4766-98ba-c3d23efcccb1/ebb995bd-0019-4c04-a0dd-2962c6aaae17"
-					(reference "#PWR032")
+					(reference "#PWR035")
 					(unit 1)
 				)
@@
 		(dnp no)
 		(fields_autoplaced yes)
-		(property "Reference" "#PWR034"
+		(property "Reference" "#PWR037"
 			(at 234.95 125.73 0)
 			(hide yes)
@@
 			(project "BMU"
 				(path "/efb70416-ce55-4766-98ba-c3d23efcccb1/ebb995bd-0019-4c04-a0dd-2962c6aaae17"
-					(reference "#PWR034")
+					(reference "#PWR037")
 					(unit 1)
 				)
@@
 		(in_pos_files yes)
 		(dnp no)
-		(property "Reference" "#PWR030"
+		(property "Reference" "#PWR033"
 			(at 201.93 124.46 0)
 			(hide yes)
@@
 			(project "BMU"
 				(path "/efb70416-ce55-4766-98ba-c3d23efcccb1/ebb995bd-0019-4c04-a0dd-2962c6aaae17"
-					(reference "#PWR030")
+					(reference "#PWR033")
 					(unit 1)
 				)
@@
 					(unit 1)
 				)
+			)
+		)
+	)
+	(symbol
+		(lib_id "Connector:TestPoint_Small")
+		(at 264.16 140.97 0)
+		(unit 1)
+		(body_style 1)
+		(exclude_from_sim no)
+		(in_bom yes)
+		(on_board yes)
+		(in_pos_files yes)
+		(dnp no)
+		(fields_autoplaced yes)
+		(property "Reference" "TP18"
+			(at 265.43 139.6999 0)
+			(show_name no)
+			(do_not_autoplace no)
+			(effects
+				(font
+					(size 1.27 1.27)
+				)
+				(justify left)
+			)
+		)
+		(property "Value" "TestPoint_Small"
+			(at 265.43 142.2399 0)
+			(hide yes)
+			(show_name no)
+			(do_not_autoplace no)
+			(effects
+				(font
+					(size 1.27 1.27)
+				)
+				(justify left)
+			)
+		)
+		(property "Footprint" "TestPoint:TestPoint_THTPad_D1.5mm_Drill0.7mm"
+			(at 269.24 140.97 0)
+			(hide yes)
+			(show_name no)
+			(do_not_autoplace no)
+			(effects
+				(font
+					(size 1.27 1.27)
+				)
+			)
+		)
+		(property "Datasheet" ""
+			(at 269.24 140.97 0)
+			(hide yes)
+			(show_name no)
+			(do_not_autoplace no)
+			(effects
+				(font
+					(size 1.27 1.27)
+				)
+			)
+		)
+		(property "Description" "test point"
+			(at 264.16 140.97 0)
+			(hide yes)
+			(show_name no)
+			(do_not_autoplace no)
+			(effects
+				(font
+					(size 1.27 1.27)
+				)
+			)
+		)
+		(pin "1"
+		)
+		(instances
+			(project "BMU"
+				(path "/efb70416-ce55-4766-98ba-c3d23efcccb1/ebb995bd-0019-4c04-a0dd-2962c6aaae17"
+					(reference "TP18")
+					(unit 1)
+				)
