File: Hardware/BMU/BMU-COM Bridge.kicad_sch (KiCad schematic)
At the start: 35 parts, among them T1 CEP99-102, T2 CEP99-102, U4 BQ79600PWRQ1, U8 PESD5V0L2BT, U9 PESD5V0L2BT

Commit message: update power part
Parts:
- renumbered C12 to C10, C22 to C11, C23 to C12, C18 to C3, C19 to C4, C20 to C5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

Commit message: finish BMU, add test point + comment
Parts:
- R12: renamed from R10; value 100k -> 10k
- renumbered R8 to R10, R9 to R11, R11 to R13, R12 to R14, R13 to R15, R14 to R16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
