File: Hardware/BMU/BMU.kicad_pcb (KiCad board)
At the start: 4 copper layers, 74 parts, among them IC1 STM32C092RCT6, J1 IN/GND, J2 HIGH SIDE, J3 I2C, J4 LOW SIDE, J5 SHUNT, J6 Conn_ARM_JTAG_SWD_10, J7 CAN, J8 AUX_IO, Q2 AO3401A, T1 CEP99-102, T2 CEP99-102, U1 TPS54202DDC, U2 TLV75533PDBV, U4 BQ79600PWRQ1, U5 MCP2562FDT-H_SN, U8 PESD5V0L2BT, U9 PESD5V0L2BT

Commit message: update power part
Parts:
- removed the C1 at (166.6, 78.7)
- removed the C2 at (166.7, 75.7)
- removed the C3 at (182.2, 77.7)
- removed the C4 at (190.3, 80.2)
- removed the C5 at (190.3, 83.6)
- removed the C6 at (190.2, 87.2)
- removed D2: BZT52-C15, Diode_SMD:D_SOD-123
- removed J7: CAN, Connector_PinHeader_2.54mm:PinHeader_1x03_P2.54mm_Vertical
- removed the J8 at (219.3, 135.7)
- removed L1: 15u, Inductor_SMD:L_7.3x7.3_H4.5
- removed Q2: AO3401A, Package_TO_SOT_SMD:SOT-23
- removed the R1 at (171.2, 76.2)
- removed the R2 at (171.2, 79.2)
- removed the R3 at (197.2, 77.7)
- removed the R4 at (197.2, 81.2)
- removed the R5 at (197.2, 84.2)
- added CR1: MMSZ5245B-7-F, MMSZ5245B-7-F:SOD123_DIO, F.Cu at (151.7, 82.0)
- added J10: ALERT, Connector_PinHeader_2.54mm:PinHeader_1x01_P2.54mm_Vertical, F.Cu at (172.0, 131.5)
- added J11: CAN, 691382000003:691382000003, F.Cu at (184.0, 99.0)
- added J12: Conn_ST_STDC14, Connector_PinHeader_1.27mm:PinHeader_2x07_P1.27mm_Vertical, F.Cu at (184.5, 112.7)
- added J13: GPIO, Connector_PinHeader_2.54mm:PinHeader_1x04_P2.54mm_Vertical, F.Cu at (185.5, 133.1)
- added J14: LED, Connector_PinHeader_2.54mm:PinHeader_1x02_P2.54mm_Vertical, F.Cu at (166.3, 131.3)
- added J4: GND, Connector_PinHeader_2.54mm:PinHeader_1x04_P2.54mm_Vertical, F.Cu at (185.0, 82.0)
- added J9: SHUNT, Connector_PinHeader_2.54mm:PinHeader_1x02_P2.54mm_Vertical, F.Cu at (155.5, 131.5)
- added Q1: DMP3099L, Package_TO_SOT_SMD:SOT-23, F.Cu at (156.7, 80.5)
- J1: renamed from J2; footprint 70551-0038:CONN_70551-xxxx_04_MOL -> 705510038:CONN_70551-xxxx_04_MOL
- J2: renamed from J4; footprint 70551-0038:CONN_70551-xxxx_04_MOL -> 705510038:CONN_70551-xxxx_04_MOL
- J3: renamed from J1; value IN/GND -> POWER
- J5: value SHUNT -> 5V; footprint Connector_PinHeader_2.54mm:PinHeader_1x03_P2.54mm_Vertical -> Connector_PinHeader_2.54mm:PinHeader_1x02_P2.54mm_Vertical
- J6: value Conn_ARM_JTAG_SWD_10 -> 3V3; footprint Connector_PinHeader_1.27mm:PinHeader_2x05_P1.27mm_Vertical -> Connector_PinHeader_2.54mm:PinHeader_1x02_P2.54mm_Vertical
- U1: value TPS54202DDC -> OKI-78SR-5_1.5-W36-C; footprint Package_TO_SOT_SMD:SOT-23-6 -> Converter_DCDC:Converter_DCDC_Murata_OKI-78SR_Vertical
- moved J5 61.4 mm to (177.5, 75.0), turned to -90 degrees
- moved J6 49.2 mm to (182.5, 88.0)
- moved R24 42.1 mm to (177.2, 94.5), turned to 180 degrees
- moved J8 39.6 mm to (161.0, 131.5), turned to 0 degrees
- moved C17 38.2 mm to (173.7, 103.5), turned to 0 degrees
- moved R23 37.9 mm to (173.8, 94.5), turned to 180 degrees
- moved C1 37.9 mm to (172.5, 80.0), turned to 90 degrees
- moved CR2 35.3 mm to (179.4, 107.1)
- moved U6 34.5 mm to (175.1, 98.5)
- moved C2 32.0 mm to (179.0, 80.0), turned to 90 degrees
- moved U2 28.0 mm to (175.6, 79.9)
- moved C16 25.3 mm to (177.2, 103.5)
- moved IC1 17.5 mm to (168.6, 116.2)
- moved C15 16.9 mm to (159.5, 111.7), turned to 180 degrees
- moved C14 16.4 mm to (159.5, 114.7), turned to 180 degrees
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- renumbered C8 to C1, C12 to C10, C22 to C11, C23 to C12, C17 to C16, C16 to C17, C7 to C2, C18 to C3, C19 to C4, C20 to C5, C10 to C6, C11 to C7, C21 to C8, CR1 to CR2, J3 to J8, R6 to R1, R8 to R10, R20 to R11, R21 to R12, R15 to R13, R22 to R14, R23 to R15, R24 to R16, R25 to R17, R26 to R18, R27 to R19, R10 to R2, R28 to R20, R29 to R21, R13 to R22, R14 to R23, R16 to R24, R11 to R3, R12 to R4, R17 to R5, R9 to R6, R18 to R7, R19 to R8, R7 to R9, U8 to U3, U9 to U5, U5 to U6
Connections:
- IC1 pad 13: unconnected-(IC1-PC0-Pad13) -> /BMU-MCU/SHUTDOWN
- IC1 pad 14: unconnected-(IC1-PC1-Pad14) -> /BMU-MCU/GPIO_SPARE1
- IC1 pad 15: unconnected-(IC1-PC2-Pad15) -> /BMU-MCU/GPIO_SPARE2
- IC1 pad 16: unconnected-(IC1-PC3-Pad16) -> /BMU-MCU/GPIO_SPARE3
- IC1 pad 19: unconnected-(IC1-PA2-Pad19) -> Net-(IC1-PA2)
- IC1 pad 20: unconnected-(IC1-PA3-Pad20) -> Net-(IC1-PA3)
- IC1 pad 30: /BMU-MCU/STATUS_LED -> /BMU-MCU/FAULT_LED
- IC1 pad 31: /BMU-MCU/SHUTDOWN_REQ -> /BMU-MCU/POWER_LED
- J5 pad 1: +3V3 -> +5V
- J5 pad 2: /BMU-MCU/ALERT_SHUNT -> +5V
- J6 pad 2: Net-(IC1-PA13) -> +3V3
- U1 pad 1: GND -> /BMU-POWER/VIN_PROTECTED
- U1 pad 2: Net-(U1-SW) -> GND
- U1 pad 3: /BMU-POWER/VIN_PROTECTED -> +5V
Routing:
- net GND: track 0.00 -> 282.9 mm
- net +3V3: track 0.00 -> 124.9 mm
- net +5V: track 0.00 -> 59.5 mm
- net /J4_CANH: track 0.00 -> 27.0 mm
- net /BMU-COM Bridge/COMLP_OPT: track 23.8 -> 0.00 mm
- net /BMU-COM Bridge/COMHN_OPT: track 23.8 -> 0.00 mm
- net /BMU-COM Bridge/COMHP_OPT: track 22.9 -> 0.00 mm
- net /BMU-COM Bridge/COMLN_OPT: track 22.8 -> 0.00 mm
- net /J4_CANL: track 0.00 -> 18.3 mm
- net /BMU-POWER/VIN_PROTECTED: track 0.00 -> 16.1 mm
- net Net-(Q1-G): track 0.00 -> 12.8 mm
- net Net-(R20-Pad2): track 7.49 -> 0.00 mm
- net Net-(R2-Pad2): track 7.24 -> 0.00 mm
- net Net-(C3-Pad1): track 6.32 -> 0.00 mm
- net +12V: track 0.00 -> 5.40 mm
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- added copper zone on F.Cu, net +12V
- added copper zone on In2.Cu, net +3V3
- added copper zone on In2.Cu, net +5V
- added copper zone on B.Cu, net GND
- added copper zone on F.Cu, net GND
- added copper zone on In1.Cu, net GND
- added copper zone on In2.Cu, net GND
Other:
- board outline added: 105 x 65.5 mm
- board text added: "VIKING MOTOR SPORTS (VMS) BATTERY MANAGEMENT UNIT (BMU) 2026.4 Capstone TEAM-12"
- board text removed: "VIKING MOTOR SPORTS (VMS) BATTERY MANAGEMENT UNIT (BMU) 2026.4"

Commit message: finish BMU, add test point + comment
Parts:
- removed J14: LED, Connector_PinHeader_2.54mm:PinHeader_1x02_P2.54mm_Vertical
- added D1: LED, LED_SMD:LED_0805_2012Metric_Pad1.15x1.40mm_HandSolder, F.Cu at (173.5, 75.5)
- added D2: LED, LED_SMD:LED_0805_2012Metric_Pad1.15x1.40mm_HandSolder, F.Cu at (177.0, 87.0)
- added D3: LED, LED_SMD:LED_0805_2012Metric_Pad1.15x1.40mm_HandSolder, F.Cu at (159.5, 109.5)
- added J8: FAULT, Connector_PinHeader_2.54mm:PinHeader_1x01_P2.54mm_Vertical, F.Cu at (166.3, 131.3)
- added R2: 1k, Resistor_SMD:R_0805_2012Metric, F.Cu at (172.0, 81.0)
- added R25: 1k, Resistor_SMD:R_0805_2012Metric, F.Cu at (159.6, 123.5)
- added R3: 1k, Resistor_SMD:R_0805_2012Metric, F.Cu at (177.1, 89.0)
- added SW1: Power Switch, Button_Switch_THT:SW_DIP_SPSTx01_Slide_9.78x4.72mm_W7.62mm_P2.54mm, F.Cu at (134.4, 75.0)
- added SW2: RESET Switch, Button_Switch_SMD:SW_Push_1P1T_NO_CK_KMR2, F.Cu at (179.0, 131.5)
- added TP1: TestPoint_Small, TestPoint:TestPoint_THTPad_D1.5mm_Drill0.7mm, F.Cu at (161.0, 91.0)
- added TP10: TestPoint_Small, TestPoint:TestPoint_THTPad_D1.5mm_Drill0.7mm, F.Cu at (181.5, 108.5)
- added TP11: TestPoint_Small, TestPoint:TestPoint_THTPad_D1.5mm_Drill0.7mm, F.Cu at (176.0, 108.5)
- added TP12: TestPoint_Small, TestPoint:TestPoint_THTPad_D1.5mm_Drill0.7mm, F.Cu at (146.0, 76.0)
- added TP13: TestPoint_Small, TestPoint:TestPoint_THTPad_D1.5mm_Drill0.7mm, F.Cu at (160.0, 84.5)
- added TP14: TestPoint_Small, TestPoint:TestPoint_THTPad_D1.5mm_Drill0.7mm, F.Cu at (151.8, 130.8)
- added TP15: TestPoint_Small, TestPoint:TestPoint_THTPad_D1.5mm_Drill0.7mm, F.Cu at (169.0, 103.0)
- added TP16: TestPoint_Small, TestPoint:TestPoint_THTPad_D1.5mm_Drill0.7mm, F.Cu at (151.5, 134.5)
- added TP17: TestPoint_Small, TestPoint:TestPoint_THTPad_D1.5mm_Drill0.7mm, F.Cu at (186.0, 92.5)
- added TP18: TestPoint_Small, TestPoint:TestPoint_THTPad_D1.5mm_Drill0.7mm, F.Cu at (178.5, 112.0)
- added TP2: TestPoint_Small, TestPoint:TestPoint_THTPad_D1.5mm_Drill0.7mm, F.Cu at (154.0, 93.0)
- added TP3: TestPoint_Small, TestPoint:TestPoint_THTPad_D1.5mm_Drill0.7mm, F.Cu at (169.0, 107.5)
- added TP4: TestPoint_Small, TestPoint:TestPoint_THTPad_D1.5mm_Drill0.7mm, F.Cu at (165.0, 106.0)
- added TP5: TestPoint_Small, TestPoint:TestPoint_THTPad_D1.5mm_Drill0.7mm, F.Cu at (154.0, 126.5)
- added TP6: TestPoint_Small, TestPoint:TestPoint_THTPad_D1.5mm_Drill0.7mm, F.Cu at (158.5, 128.5)
- added TP7: TestPoint_Small, TestPoint:TestPoint_THTPad_D1.5mm_Drill0.7mm, F.Cu at (185.5, 108.0)
- added TP8: TestPoint_Small, TestPoint:TestPoint_THTPad_D1.5mm_Drill0.7mm, F.Cu at (170.0, 87.5)
- added TP9: TestPoint_Small, TestPoint:TestPoint_THTPad_D1.5mm_Drill0.7mm, F.Cu at (170.5, 93.0)
- R12: renamed from R10; value 100k -> 10k
- moved CR2 14.6 mm to (180.5, 92.5), turned to 90 degrees
- moved R8 5.90 mm to (157.6, 92.0), turned to 180 degrees
- moved U1 4.11 mm to (161.9, 78.5), turned to 0 degrees
- moved C16 3.67 mm to (173.6, 103.5), turned to 180 degrees
- moved C17 3.33 mm to (177.1, 103.5), turned to 180 degrees
- moved R11 3.10 mm to (157.6, 95.0), turned to 180 degrees
- moved R12 3.10 mm to (157.5, 98.0), turned to 180 degrees
- moved F1 3.01 mm to (149.0, 80.0), turned to 90 degrees
- moved U2 2.24 mm to (177.5, 81.1), turned to -90 degrees
- moved CR1 2.14 mm to (152.5, 80.0), turned to 90 degrees
- moved C1 1.85 mm to (174.0, 81.0), turned to -90 degrees
- moved C2 1.85 mm to (180.5, 81.0)
- moved J6 1.58 mm to (179.0, 75.5)
- moved J13 1.15 mm to (184.5, 111.5)
- moved J12 0.91 mm to (184.0, 99.9)
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- renumbered J9 to J10, J10 to J11, J11 to J12, J12 to J13, J13 to J4, J4 to J5, J5 to J6, J6 to J7, J8 to J9, R8 to R10, R9 to R11, R11 to R13, R12 to R14, R13 to R15, R14 to R16, R15 to R17, R16 to R18, R17 to R19, R18 to R20, R19 to R21, R20 to R22, R21 to R23, R22 to R24, R23 to R26, R24 to R27, R2 to R4, R3 to R5, R4 to R6, R5 to R7, R6 to R8, R7 to R9
Connections:
- C13 pad 1: Net-(IC1-PF2-NRST) -> GND
- C13 pad 2: GND -> Net-(IC1-PF2-NRST)
- F1 pad 1: +12V -> Net-(SW1-A)
- F1 pad 2: Net-(Q1-D) -> +12V
- IC1 pad 31: /BMU-MCU/POWER_LED -> unconnected-(IC1-PB11-Pad31)
- J13 pad 12: GND -> Net-(IC1-PF2-NRST)
Routing:
- net GND: track 282.9 -> 121.3 mm, vias 0 -> 14
- net +3V3: track 124.9 -> 41.6 mm, vias 0 -> 7
- net Net-(IC1-PF2-NRST): track 0.00 -> 54.9 mm
- net /BMU-MCU/ALERT_SHUNT: track 0.00 -> 49.3 mm
- net /BMU-COM Bridge/MOSI/RX: track 0.00 -> 37.4 mm, vias 0 -> 2
- net /BMU-MCU/SHUTDOWN: track 0.00 -> 35.2 mm, vias 0 -> 1
- net /SCL_STM32: track 0.00 -> 32.3 mm, vias 0 -> 1
- net /BMU-COM Bridge/FAULT_N: track 0.00 -> 30.3 mm, vias 0 -> 2
- net /BMU-COM Bridge/MISO/TX: track 0.00 -> 29.9 mm, vias 0 -> 2
- net /SDA_STM32: track 0.00 -> 29.8 mm, vias 0 -> 1
- net COMHP: track 0.00 -> 27.3 mm, vias 0 -> 2
- net /BMU-MCU/GPIO_SPARE3: track 0.00 -> 27.1 mm, vias 0 -> 1
- net /BMU-MCU/GPIO_SPARE2: track 0.00 -> 26.2 mm, vias 0 -> 1
- net COMLP: track 0.00 -> 26.1 mm, vias 0 -> 2
- net /BMU-CAN/CAN_STBY: track 0.00 -> 25.9 mm
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- removed copper zone on F.Cu, net +12V
