File: Hardware/BMU/BMU.kicad_sch (KiCad schematic)
At the start: 7 parts, among them J1 IN/GND, J2 HIGH SIDE, J3 I2C, J4 LOW SIDE, J5 SHUNT, J7 CAN, J8 AUX_IO

Commit message: update power part
Parts:
- removed J5: SHUNT, Connector_PinHeader_2.54mm:PinHeader_1x03_P2.54mm_Vertical, symbol Connector_Generic:Conn_01x03
- removed J7: CAN, Connector_PinHeader_2.54mm:PinHeader_1x03_P2.54mm_Vertical, symbol Connector_Generic:Conn_01x03
- removed J8: AUX_IO, Connector_PinHeader_2.54mm:PinHeader_1x02_P2.54mm_Vertical, symbol Connector_Generic:Conn_01x02
- added J10: ALERT, Connector_PinHeader_2.54mm:PinHeader_1x01_P2.54mm_Vertical, symbol Connector_Generic:Conn_01x01
- added J11: CAN, 691382000003:691382000003, symbol 691382000003:691382000003
- added J13: GPIO, Connector_PinHeader_2.54mm:PinHeader_1x04_P2.54mm_Vertical, symbol Connector_Generic:Conn_01x04
- added J14: LED, Connector_PinHeader_2.54mm:PinHeader_1x02_P2.54mm_Vertical, symbol Connector_Generic:Conn_01x02
- added J4: GND, Connector_PinHeader_2.54mm:PinHeader_1x04_P2.54mm_Vertical, symbol Connector_Generic:Conn_01x04
- added J5: 5V, Connector_PinHeader_2.54mm:PinHeader_1x02_P2.54mm_Vertical, symbol Connector_Generic:Conn_01x02
- added J6: 3V3, Connector_PinHeader_2.54mm:PinHeader_1x02_P2.54mm_Vertical, symbol Connector_Generic:Conn_01x02
- added J9: SHUNT, Connector_PinHeader_2.54mm:PinHeader_1x02_P2.54mm_Vertical, symbol Connector_Generic:Conn_01x02
- J1: renamed from J2; footprint CONN_70551-xxxx_04_MOL -> 705510038:CONN_70551-xxxx_04_MOL
- J2: renamed from J4; footprint CONN_70551-xxxx_04_MOL -> 705510038:CONN_70551-xxxx_04_MOL
- J3: renamed from J1; value IN/GND -> POWER
- renumbered J3 to J8
Connections:
- net BMU-MCU/3V3_SHUNT: now also J9.2 (Pin_2)
- net BMU-MCU/ALERT_SHUNT: now also J10.1 (Pin_1)
- net BMU-MCU/GND_SHUNT: now also J9.1 (Pin_1)
- net J4_CANH: now also J11.1
- net J4_CANL: now also J11.2
- net J4_GND: now also J11.3
- new net BMU-MCU/FAULT_LED: J14.1 (Pin_1)
- new net BMU-MCU/GPIO_SPARE1: J13.4 (Pin_4)
- new net BMU-MCU/GPIO_SPARE2: J13.3 (Pin_3)
- new net BMU-MCU/GPIO_SPARE3: J13.2 (Pin_2)
- new net BMU-MCU/POWER_LED: J14.2 (Pin_2)
- new net BMU-MCU/SHUTDOWN: J13.1 (Pin_1)
- new net BMU-POWER/3V3: J6.1 (Pin_1), J6.2 (Pin_2)
- new net BMU-POWER/5V: J5.1 (Pin_1), J5.2 (Pin_2)
- new net BMU-POWER/GND: J4.1 (Pin_1), J4.2 (Pin_2), J4.3 (Pin_3), J4.4 (Pin_4)
Other:
- sheet BMU-MCU ports: added FAULT_LED, GPIO_SPARE1, GPIO_SPARE2, GPIO_SPARE3, POWER_LED, SHUTDOWN, UART1_RX, UART1_TX; removed SHUTDOWN_REQ, STATUS_LED, UART_RX, UART_TX
- sheet BMU-POWER ports: added 3V3, 5V, GND; removed none
- moved on the sheet: J2

Commit message: finish BMU, add test point + comment
Parts:
- removed J14: LED, Connector_PinHeader_2.54mm:PinHeader_1x02_P2.54mm_Vertical, symbol Connector_Generic:Conn_01x02
- added J8: FAULT, Connector_PinHeader_2.54mm:PinHeader_1x01_P2.54mm_Vertical, symbol Connector_Generic:Conn_01x01
- added TP1, TP10, TP11, TP2, TP3, TP4, TP5, TP6, TP7, TP8, TP9: TestPoint_Small, TestPoint:TestPoint_THTPad_D1.5mm_Drill0.7mm, symbol Connector:TestPoint_Small
- renumbered J9 to J10, J10 to J11, J11 to J12, J13 to J4, J4 to J5, J5 to J6, J6 to J7, J8 to J9
Connections:
- net BMU-CAN/CAN_RX: now also TP10.1
- net BMU-CAN/CAN_STBY: now also TP9.1
- net BMU-CAN/CAN_TX: now also TP11.1
- net BMU-COM Bridge/FAULT_N: now also TP3.1
- net BMU-COM Bridge/MISO/TX: now also TP2.1
- net BMU-COM Bridge/MOSI/RX: now also TP1.1
- net BMU-MCU/3V3_SHUNT: now also TP7.1
- net BMU-MCU/ALERT_SHUNT: now also TP4.1
- net BMU-MCU/FAULT_LED: now also J8.1 (Pin_1)
- net BMU-MCU/GND_SHUNT: now also TP8.1
- net SCL_STM32: now also TP6.1
- net SDA_STM32: now also TP5.1
Other:
- sheet BMU-MCU ports: added none; removed POWER_LED
- note added: "BMU TOP-LEVEL ARCHITECTURE This page summarizes the BMU interface board, including power distribution, STM32 control, BQ79600 battery-monitor communication, CAN-FD interface, shunt-board interface, external connectors, and debug/test access points. 1. POWER J3 receives the 12 V BMU input. BMU-POWER provides fuse protection, power switch, PMOS input protection, 12 V to 5 V conversion, 5 V to 3.3 V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"
- note removed: "1. BMU-POWER Core function: Conditions the 12 V input and generates the regulated 5 V and 3.3 V rails. Short version for page 1: 12 V input conditioning and protection Generates 5 V and 3.3 V rails Supplies power to BMU circuits"
- note removed: "2. BMU-BQ79600 Core function: Implements the isolated BQ79600 host bridge between the MCU and the external battery-monitor daisy-chain / ring network. Short version for page 1: Isolated BQ79600 host bridge interface Connects STM32 to external battery monitor chain Handles daisy-chain / ring communication"
- note removed: "3. BMU-MCU Core function: Main STM32 controller for BMU logic, diagnostics, and communications. Short version for page 1: Main STM32 control page Executes BMU control and monitoring logic Interfaces with BQ, CAN, and external shunt board"
- note removed: "4. BMU-CAN Core function: Provides the physical CAN-FD bus interface between the BMU and vehicle ECU. Short version for page 1: CAN-FD transceiver interface Converts MCU signals to CAN bus levels Connects BMU to ECU / vehicle network"
- note removed: "Optional module, if you keep it later 5. BMU-SAFETY Core function: Routes BMU fault and status signals to external shutdown or safety circuits. Short version for page 1: Safety / shutdown interface Routes fault and status signals Optional external safety path"
- moved on the sheet: J1, J10, J11, J12, J2, J3, J4, J5, J6, J7, J9
