File: Hardware/Monitor/Montior.kicad_sch (KiCad schematic)
At the start: 94 parts, among them J15? Conn_01x22

Commit message: Update monitor hardware files
Parts:
- removed J?: Daisy-chain communication pins, symbol Connector_Generic:Conn_01x04
- added C42, C43, C44, C45, C46, C47: 100pF, Capacitor_SMD:C_0805_2012Metric, symbol Device:C
- added J3, J4: 705510038, footprints7055:CONN_70551-xxxx_04_MOL, symbol 2026-04-25_22-53-02:705510038
- added R41, R42: 10.0k, Resistor_SMD:R_0805_2012Metric, symbol Device:R_US
- added R45, R46, R47, R48, R53, R54, R55, R56: 0, Resistor_SMD:R_0805_2012Metric, symbol Device:R_US
- added R49, R50, R57, R58: 51, Resistor_SMD:R_0805_2012Metric, symbol Device:R_US
- added R51, R52, R59, R60: 499, Resistor_SMD:R_0805_2012Metric, symbol Device:R_US
- added RT7, RT8: T*, Connector_PinHeader_1.00mm:PinHeader_1x02_P1.00mm_Vertical, symbol Connector_Generic:Conn_02x01
- added T1, T3: CEP99-102, KiCadCEP99:CEP99102, symbol CEP99-102:CEP99-102
- added U3, U4: PESD5V0L2BT, footprintspes:SOT23_NEX, symbol 2026-03-31_20-22-46:PESD5V0L2BT
- C1, C10, C11, C12, C13, C14, C15, C16, C17, C18, C19, C2, C20, C21, C22, C23, C24, C25, C26, C27, C28, C29, C3, C30, C31, C32, C33, C34, C35, C36, C37, C38, C39, C4, C40, C41, C5, C6, C7, C8, C9: footprint (none) -> Capacitor_SMD:C_0805_2012Metric
- J1: renamed from J15?; footprint (none) -> Connector_PinHeader_1.00mm:PinHeader_1x22_P1.00mm_Vertical
- J2: renamed from J?; footprint (none) -> Connector_PinHeader_1.00mm:PinHeader_1x02_P1.00mm_Vertical
- Q1: renamed from Q?; footprint (none) -> ZXTN4004KTC:TO-252
- R1, R10, R11, R12, R13, R14, R15, R16, R17, R18, R19, R2, R20, R21, R22, R23, R24, R25, R26, R27, R28, R29, R3, R30, R31, R32, R33, R34, R35, R36, R37, R38, R39, R4, R40, R5, R6, R7, R8, R9: footprint (none) -> Resistor_SMD:R_0805_2012Metric
- R43: renamed from R41; footprint (none) -> Resistor_SMD:R_0805_2012Metric
- R44: renamed from R42; footprint (none) -> Resistor_SMD:R_0805_2012Metric
- RT1, RT2, RT3, RT4, RT5, RT6: footprint (none) -> Connector_PinHeader_1.00mm:PinHeader_1x02_P1.00mm_Vertical
- U1: renamed from U?; footprint Snapeda:PAP0064F-IPC_A -> pq_footprints:PAP0064F-IPC_A
Connections:
- net CEL13 is gone; now on net CELL13: R27.1, R28.1
- net CELL16 is gone; now on net CELL16S: R33.1, R34.1
- net CB12: no longer U1.2 (CB16), U1.4 (CB15), U1.6 (CB14), U1.8 (CB13)
- net CB13: now also U1.8 (CB13)
- net CB14: now also U1.6 (CB14)
- net CB15: now also U1.4 (CB15)
- net CB16: now also U1.2 (CB16)
- net CELL0: now also J1.1 (Pin_1), J1.21 (Pin_21), J1.22 (Pin_22), J1.3 (Pin_3)
- net CELL0S: now also J1.4 (Pin_4)
- net CELL1: now also J1.5 (Pin_5)
- net CELL10: now also J1.14 (Pin_14)
- net CELL11: now also J1.15 (Pin_15)
- net CELL12: now also J1.16 (Pin_16); no longer R44.1, U1.1 (BAT)
- net CELL13: now also J1.17 (Pin_17)
- net CELL14: now also J1.18 (Pin_18)
- net CELL15: now also J1.19 (Pin_19)
- net CELL16S: now also J1.20 (Pin_20)
- net CELL2: now also J1.6 (Pin_6)
- net CELL3: now also J1.7 (Pin_7)
- net CELL4: now also J1.8 (Pin_8)
- net CELL5: now also J1.9 (Pin_9)
- net CELL6: now also J1.10 (Pin_10)
- net CELL7: now also J1.11 (Pin_11)
- net CELL8: now also J1.12 (Pin_12)
- net CELL9: now also J1.13 (Pin_13)
- net GND: now also C42.2, C43.2, C44.2, C45.2, C46.2, C47.2, R51.2, R52.1, R59.2, R60.1, RT7.2 (Pin_2), RT8.2 (Pin_2), U3.3, U4.3
- net GPIO7: now also R41.2, RT7.1 (Pin_1)
- net GPIO8: now also R42.2, RT8.1 (Pin_1)
- net RX: now also U1.45 (CVDD), U1.52 (RX)
- net TSREF: now also R41.1, R42.1
- net VC12: no longer U1.3 (VC16), U1.5 (VC15), U1.7 (VC14), U1.9 (VC13)
- net VC13: now also U1.9 (VC13)
- net VC14: now also U1.7 (VC14)
- net VC15: now also U1.5 (VC15)
- net VC16: now also U1.3 (VC16)
- net COMLP: now reaches U1.40 (COMLP)
- net COMLP: now also C44.1, R49.2, R51.1
- net COMLN: now reaches U1.41 (COMLN)
- net COMLN: now also C43.1, R50.2, R52.2
- net COMHN: now reaches U1.42 (COMHN)
- net COMHN: now also C46.1, R58.2, R60.2
- net COMHP: now reaches U1.43 (COMHP)
- net COMHP: now also C47.1, R57.2, R59.1
- net PWR: now reaches J1.2 (Pin_2)
- net PWR: now also R44.1, U1.1 (BAT)
- new net: R47.1, T1.5
- new net: C45.1, T3.2, T3.3
- new net: R56.1, T3.1
- new net: R55.1, T3.4
- new net: R53.2, T3.5
- new net: T3.6, T3.7
- new net: R54.2, T3.8
- new net: R46.2, T1.1
- new net: R48.1, T1.8
- new net: R45.2, T1.4
- new net: C42.1, T1.6, T1.7
- new net: T1.2, T1.3
- new net COMHN_OPT: R56.2, R58.1, U4.2
- new net COMHP_OPT: R55.2, R57.1, U4.1
- new net COMLN_OPT: R48.2, R50.1, U3.1
- new net COMLP_OPT: R47.2, R49.1, U3.2
- new net ISO COMHN: J4.4, R54.1
- new net ISO COMHP: J4.3, R53.1
- new net ISO COMLN: J3.1, R46.1
- new net ISO COMLP: J3.2, R45.1
- no-connect marks 4 -> 8
Other:
- moved on the sheet: C1, C10, C11, C12, C13, C14, C15, C16, C17, C18, C19, C2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
