File: Hardware/Battery Management Unit (BMU)/BMU-CAN.kicad_sch (KiCad schematic)
At the start: 8 parts, among them U6 MCP2562FDT-H_SN

Commit message: Both boards are now fully completed: the BMU and CMU.
Parts:
- TP17, TP18: symbol Connector:TestPoint_Small -> Connector:TestPoint_Square
Changed lines of the file:
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@@
 	)
 	(symbol
-		(lib_id "Connector:TestPoint_Small")
+		(lib_id "Connector:TestPoint_Square")
 		(at 264.16 135.89 0)
 		(unit 1)
@@
 		(in_pos_files yes)
 		(dnp no)
-		(fields_autoplaced yes)
 		(property "Reference" "TP17"
-			(at 265.43 134.6199 0)
+			(at 265.938 134.366 0)
 			(show_name no)
 			(do_not_autoplace no)
@@
 			)
 		)
-		(property "Datasheet" ""
+		(property "Datasheet" "~"
 			(at 269.24 135.89 0)
 			(hide yes)
@@
 	)
 	(symbol
-		(lib_id "Connector:TestPoint_Small")
+		(lib_id "Connector:TestPoint_Square")
 		(at 264.16 140.97 0)
 		(unit 1)
@@
 		(in_pos_files yes)
 		(dnp no)
-		(fields_autoplaced yes)
 		(property "Reference" "TP18"
-			(at 265.43 139.6999 0)
+			(at 265.938 139.7 0)
 			(show_name no)
 			(do_not_autoplace no)
@@
 			)
 		)
-		(property "Datasheet" ""
+		(property "Datasheet" "~"
 			(at 269.24 140.97 0)
 			(hide yes)
