File: Hardware/Battery Management Unit (BMU)/Battery Management Unit (BMU).kicad_pcb (KiCad board)
At the start: 4 copper layers, 105 x 66 mm, 90 parts, among them IC1 STM32C092RCT6, J1 HIGH SIDE, J10 SHUNT, J11 Conn_ST_STDC14, J2 LOW SIDE, J3 POWER, J4 GPIO, J5 5V, J6 3V3, J7 GND, J8 pin header, J9 CAN, Q1 DMP3099L, SW1 Power Switch, SW2 SW_Push, T1 CEP99-102, T2 CEP99-102, U1 OKI-78SR-5_1.5-W36-C, U2 TLV75533PDBV, U3 PESD5V0L2BT, U4 BQ79600PWRQ1, U5 PESD5V0L2BT, U6 MCP2562FDT-H_SN

Commit message: doubled up pin for bmu
Parts:
- D1, D2: value LED -> GRN
- J10: footprint Connector_PinHeader_2.54mm:PinHeader_1x05_P2.54mm_Vertical -> Connector_PinHeader_2.54mm:PinHeader_1x10_P2.54mm_Vertical
- J3: footprint Connector_PinHeader_2.54mm:PinHeader_1x02_P2.54mm_Vertical -> Connector_PinHeader_2.54mm:PinHeader_1x04_P2.54mm_Vertical
- moved J4 20.7 mm to (145.4, 134.0), turned to 90 degrees
- moved TP9 12.0 mm to (139.0, 134.0)
- moved J10 10.8 mm to (162.7, 134.0)
- moved TP4 6.02 mm to (170.0, 130.5)
- moved SW1 5.70 mm to (128.9, 76.5)
- moved TP11 5.52 mm to (165.0, 130.5)
- moved TP5 4.03 mm to (175.0, 130.5)
- moved J3 2.54 mm to (152.0, 74.0), turned to -90 degrees
- moved TP7 2.24 mm to (144.5, 77.5)
- moved TP6 2.06 mm to (180.0, 130.5)
- renumbered C9 to C10, C7 to C11, C6 to C12, C12 to C4, C11 to C5, C4 to C6, C8 to C7, C5 to C8, C10 to C9, J8 to J5, J9 to J6, J5 to J7, J6 to J8, J7 to J9, R20 to R10, R7 to R11, R18 to R12, R19 to R13, R10 to R14, R11 to R15, R13 to R18, R14 to R19, R15 to R20, R12 to R21, R9 to R22, R8 to R23, R22 to R4, R23 to R5, R4 to R6, R5 to R7, R6 to R8, R21 to R9, U5 to U3, U3 to U4, U4 to U5
Connections:
- net COMHN renamed /BMU-COM Bridge/COMHN
- net COMHP renamed /BMU-COM Bridge/COMHP
- net COMLN renamed /BMU-COM Bridge/COMLN
- net COMLP renamed /BMU-COM Bridge/COMLP
- J10 pad 2: /I2C_SDA -> +3V3
- J10 pad 3: /I2C_SCL -> /I2C_SDA
- J10 pad 4: /ALERT_SHUNT -> /I2C_SDA
- J10 pad 5: GND -> /I2C_SCL
- J3 pad 1: +12V -> GND
- J4 pad 1: /BMU-MCU/GPIO_SPARE1 -> GND
- J4 pad 2: /BMU-MCU/GPIO_SPARE2 -> /BMU-MCU/SHUTDOWN
- J4 pad 4: /BMU-MCU/SHUTDOWN -> /BMU-MCU/GPIO_SPARE2
- J4 pad 5: GND -> /BMU-MCU/GPIO_SPARE1
Routing:
- net Net-(Q1-D): track 18.0 -> 22.9 mm
- net Net-(SW1-A): track 17.3 -> 22.1 mm
- net +3V3: track 27.1 -> 22.3 mm, vias 16 -> 15
- net /BMU-MCU/SHUTDOWN: track 20.2 -> 24.7 mm
- net +12V: track 7.75 -> 12.2 mm
- net /BMU-MCU/GPIO_SPARE3: track 17.1 -> 21.0 mm
- net /BMU-MCU/GPIO_SPARE2: track 17.2 -> 21.1 mm
- net /BMU-MCU/GPIO_SPARE1: track 18.1 -> 21.1 mm
- net /ALERT_SHUNT: track 30.4 -> 31.5 mm
- net /I2C_SCL: track 29.6 -> 30.5 mm

Commit message: finish! update bmu layout+BOM
Parts:
- added REF**: MountingHole_3.2mm_M3, MountingHole:MountingHole_3.2mm_M3, F.Cu at (185.0, 138.5)
- added REF**: MountingHole_3.2mm_M3, MountingHole:MountingHole_3.2mm_M3, F.Cu at (90.5, 138.5)
- added REF**: MountingHole_3.2mm_M3, MountingHole:MountingHole_3.2mm_M3, F.Cu at (185.0, 69.5)
- added REF**: MountingHole_3.2mm_M3, MountingHole:MountingHole_3.2mm_M3, F.Cu at (90.5, 69.5)
- C12, C9: value 0.1u -> 100n
- Q1: value DMP3099L -> AO3401A
- T1, T2: value CEP99-102 -> HM2147NLT; footprint Footprints:CEP99102 -> Footprints:HM2147NLT
- moved T1 28.1 mm to (112.9, 90.5), turned to -90 degrees
- moved T2 27.9 mm to (112.9, 117.5), turned to -90 degrees
- moved R7 6.51 mm to (102.5, 120.0), turned to 90 degrees
- moved R5 6.46 mm to (102.5, 88.6), turned to -90 degrees
- moved C3 4.62 mm to (123.9, 118.4)
- moved C4 4.62 mm to (123.9, 89.8)
- moved R10 4.62 mm to (123.9, 86.2)
- moved R11 4.62 mm to (123.9, 121.9)
- moved R8 4.62 mm to (123.9, 114.9)
- moved R9 4.62 mm to (123.9, 93.2)
- moved J2 3.04 mm to (100.0, 121.1)
- moved J1 3.03 mm to (100.0, 94.6)
- moved R4 2.71 mm to (102.5, 92.0), turned to 90 degrees
- moved R6 2.61 mm to (102.5, 116.5), turned to 90 degrees
- moved TP11 2.12 mm to (163.5, 129.0)
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Connections:
- C3 pad 1: Net-(C3-Pad1) -> Net-(T2-SEC_2)
- C4 pad 1: Net-(C4-Pad1) -> Net-(T1-SEC_2)
- R10 pad 1: Net-(R10-Pad1) -> Net-(T1-SEC_3)
- R11 pad 1: Net-(R11-Pad1) -> Net-(T2-SEC_3)
- R4 pad 2: Net-(R4-Pad2) -> Net-(T1-PRI_1)
- R5 pad 2: Net-(R5-Pad2) -> Net-(T1-PRI_3)
- R6 pad 2: Net-(R6-Pad2) -> Net-(T2-PRI_1)
- R7 pad 2: Net-(R7-Pad2) -> Net-(T2-PRI_3)
- R8 pad 1: Net-(R8-Pad1) -> Net-(T2-SEC_1)
- R9 pad 1: Net-(R9-Pad1) -> Net-(T1-SEC_1)
- T1 pad 1: Net-(R7-Pad2) -> Net-(T1-PRI_1)
- T1 pad 2: Net-(T1-Pad2) -> unconnected-(T1-PRI_2-Pad2)
- T1 pad 3: Net-(T1-Pad2) -> Net-(T1-PRI_3)
- T1 pad 4: Net-(R6-Pad2) -> Net-(T1-SEC_1)
- T1 pad 5: Net-(R11-Pad1) -> Net-(T1-SEC_2)
- T1 pad 6: Net-(C3-Pad1) -> Net-(T1-SEC_3)
- T2 pad 1: Net-(R9-Pad1) -> Net-(T2-PRI_1)
- T2 pad 2: Net-(C4-Pad1) -> unconnected-(T2-PRI_2-Pad2)
- T2 pad 3: Net-(C4-Pad1) -> Net-(T2-PRI_3)
- T2 pad 4: Net-(R10-Pad1) -> Net-(T2-SEC_1)
- T2 pad 5: Net-(R4-Pad2) -> Net-(T2-SEC_2)
- T2 pad 6: Net-(T2-Pad6) -> Net-(T2-SEC_3)
Routing:
- net Net-(T2-SEC_3): track 0.00 -> 12.5 mm
- net Net-(T1-PRI_3): track 0.00 -> 12.3 mm
- net Net-(T2-SEC_1): track 0.00 -> 8.42 mm
- net Net-(R4-Pad2): track 6.39 -> 0.00 mm
- net Net-(R6-Pad2): track 6.37 -> 0.00 mm
- net Net-(C4-Pad1): track 6.32 -> 0.00 mm
- net Net-(C3-Pad1): track 6.32 -> 0.00 mm
- net /LOW COMLN: track 8.62 -> 2.55 mm
- net /High COMHN: track 8.79 -> 2.75 mm
- net /BMU-COM Bridge/COMLP_OPT: track 22.9 -> 18.3 mm
- net /BMU-COM Bridge/COMLN_OPT: track 21.9 -> 17.3 mm
- net /BMU-COM Bridge/COMHP_OPT: track 22.0 -> 17.4 mm
- net /BMU-COM Bridge/COMHN_OPT: track 22.9 -> 18.3 mm
- net Net-(T1-PRI_1): track 0.00 -> 4.51 mm
- net /BMU-POWER/VIN_PROTECTED: track 14.2 -> 18.5 mm
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Other:
- board size 105 x 66 mm -> 102 x 76 mm

Commit message: add jumper+ change SW for bmu
Parts:
- removed SW1: Power Switch, Button_Switch_THT:SW_DIP_SPSTx01_Slide_9.78x4.72mm_W7.62mm_P2.54mm
- added S1: 100SP1T1B4M2QE, Footprints:SW_100SP1T1B4M2QE, F.Cu at (125.0, 76.5)
- moved TP7 9.43 mm to (136.5, 72.5)
- moved F1 5.39 mm to (144.0, 78.0), turned to 0 degrees
- moved J3 1.80 mm to (150.5, 73.0)
Routing:
- net Net-(Q1-D): track 22.7 -> 29.5 mm
- net +12V: track 11.6 -> 14.1 mm
- net Net-(F1-Pad1): track 22.1 -> 19.7 mm
- net GND: track 20.4 -> 19.1 mm

Commit message: Polishing, BOM fixes, stitching
Routing:
- net GND: vias 47 -> 84
