File: Hardware/Battery Management Unit (BMU)/Battery Management Unit (BMU).kicad_sch (KiCad schematic)
At the start: 16 parts, among them J1 HIGH SIDE, J10 SHUNT, J2 LOW SIDE, J3 POWER, J4 GPIO, J5 pin header, J6 CAN, J7 5V, J8 3V3, J9 GND

Commit message: Polishing, BOM fixes, stitching
Parts:
- TP1, TP2, TP3, TP4, TP5, TP6: now left out of the parts list
Changed lines of the file:
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@@
 	(title_block
 		(title "BATTERY MANAGEMENT UNIT (BMU)")
-		(date "2026-04-06")
+		(date "2026-06-02")
 		(rev "1.0")
 		(company "VIKING MOTOR SPORTS (VMS)")
@@
 		(body_style 1)
 		(exclude_from_sim no)
-		(in_bom yes)
+		(in_bom no)
 		(on_board yes)
 		(in_pos_files yes)
@@
 		(body_style 1)
 		(exclude_from_sim no)
-		(in_bom yes)
+		(in_bom no)
 		(on_board yes)
 		(in_pos_files yes)
@@
 		(body_style 1)
 		(exclude_from_sim no)
-		(in_bom yes)
+		(in_bom no)
 		(on_board yes)
 		(in_pos_files yes)
@@
 		(body_style 1)
 		(exclude_from_sim no)
-		(in_bom yes)
+		(in_bom no)
 		(on_board yes)
 		(in_pos_files yes)
@@
 		(body_style 1)
 		(exclude_from_sim no)
-		(in_bom yes)
+		(in_bom no)
 		(on_board yes)
 		(in_pos_files yes)
@@
 		(body_style 1)
 		(exclude_from_sim no)
-		(in_bom yes)
+		(in_bom no)
 		(on_board yes)
 		(in_pos_files yes)
