File: Hardware/Cell Monitoring Unit (CMU)/Cell Monitoring Unit (CMU).kicad_sch (KiCad schematic)
At the start: 167 parts, among them J1 TEST, J10 NTC-5, J11 NTC-6, J12 NTC-7, J13 NTC-8, J2 LOW SIDE, J3 12S, J4 705550056, J5 HIGH SIDE, J6 NTC-1, J7 NTC-2, J8 NTC-3, J9 NTC-4, T1 CEP99-102, T2 CEP99-102, U1 PESD5V0L2BT, U2 PESD5V0L2BT, U3 ZXTN4004KQTC, U4 PBQ79616PAPTQ1

Commit message: update CMU
Parts:
- J2, J5: footprint 705510038:CONN_70551-xxxx_04_MOL -> Footprints:705510038
- J4: footprint Molex 0705550056:CONN_705550000-SD_22_MOL -> Footprints:705550056
- T1, T2: footprint CEP99-102:CEP99102 -> Footprints:CEP99102
- U1, U2: footprint PESD5V0L2BT:SOT23_NEX -> Footprints:SOT23_NEX
- U3: footprint ZXTN4004KTC:DPAK_04KQTC_DIO -> Footprints:DPAK_04KQTC_DIO
- U4: footprint BQ79616PAPRQ1:PAP0064F-IPC_A -> Footprints:PAP0064F-IPC_A
- renumbered C43 to C42, C44 to C43, C45 to C44, C46 to C45, C47 to C46, C42 to C47, R49 to R47, R47 to R48, R48 to R49, R52 to R50, R53 to R51, R54 to R52, R50 to R53, R51 to R54
Other:
- note added: "BAT_TOP provides the stack-powered input for the BQ79616."
- note added: "BQ79616 External NPN Power Path"
- note added: "CELL0 is the local cell-stack reference for the CMU, not chassis ground."
- note added: "Cell connector follows the TI EVM-style sensing structure. CELL0/CELL16 are stack endpoints; CELL0S/CELL16S are sense lines."
- note added: "GPIO1–GPIO8 are routed to NTC headers for external temperature sensing."
- note added: "TSREF provides the NTC bias reference."
- note added: "Tranformer Isolation For COM Communication"
- note added: "VC inputs use 100Ω series resistors and 0.47uF capacitors to CELL0 for filtering."

Commit message: Fixed all missing symbol and footprint libraries
Parts:
- J2, J5: symbol 70551-0038:705510038 -> 705510038:705510038
- J4: symbol Molex 0705550056:705550056 -> 705550056:705550056
- U1, U2: symbol 2026-03-31_20-22-46:PESD5V0L2BT -> PESD5V0L2BT:PESD5V0L2BT
- U3: symbol ZXTN4004KTC:ZXTN4004KQTC -> ZXTN4004KQTC:ZXTN4004KQTC
- U4: symbol Snapeda:PBQ79616PAPTQ1 -> BQ79616PAPRQ1:BQ79616PAPRQ1
Changed lines of the file:
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@@
 	)
 	(symbol
-		(lib_id "2026-03-31_20-22-46:PESD5V0L2BT")
+		(lib_id "PESD5V0L2BT:PESD5V0L2BT")
 		(at 341.63 354.33 270)
 		(unit 1)
@@
 	)
 	(symbol
-		(lib_id "Snapeda:PBQ79616PAPTQ1")
+		(lib_id "BQ79616PAPRQ1:BQ79616PAPRQ1")
 		(at 435.61 217.17 0)
 		(unit 1)
@@
 				(font
 					(size 1.27 1.27)
+					(italic yes)
 				)
 			)
@@
 				(font
 					(size 1.27 1.27)
+					(italic yes)
 				)
 			)
@@
 	)
 	(symbol
-		(lib_id "70551-0038:705510038")
+		(lib_id "705510038:705510038")
 		(at 82.55 331.47 180)
 		(unit 1)
@@
 	)
 	(symbol
-		(lib_id "ZXTN4004KTC:ZXTN4004KQTC")
+		(lib_id "ZXTN4004KQTC:ZXTN4004KQTC")
 		(at 363.22 96.52 180)
 		(unit 1)
@@
 	)
 	(symbol
-		(lib_id "2026-03-31_20-22-46:PESD5V0L2BT")
+		(lib_id "PESD5V0L2BT:PESD5V0L2BT")
 		(at 193.04 359.41 270)
 		(unit 1)
@@
 	)
 	(symbol
-		(lib_id "70551-0038:705510038")
+		(lib_id "705510038:705510038")
 		(at 440.69 323.85 0)
 		(unit 1)
@@
 	)
 	(symbol
-		(lib_id "Molex 0705550056:705550056")
+		(lib_id "705550056:705550056")
 		(at 275.59 185.42 0)
 		(unit 1)

Commit message: Big schematic cleanup - made into hierarchical schematic, lots of checking on power, more text notes.
Parts:
- removed C1, C10, C11, C12, C13, C14, C15, C16, C17, C18, C2, C20, C21, C22, C23, C24, C25, C26, C27, C28, C3, C30, C31, C32, C33, C34, C35, C36, C37, C4, C5, C6, C7, C8, C9: 0.47uF, Capacitor_SMD:C_0805_2012Metric, symbol Device:C_Small
- removed C19, C29, C38, C39, C40, C47: 100pF, Capacitor_SMD:C_0805_2012Metric, symbol Device:C
- removed C41, C48: 1u, Capacitor_SMD:C_0805_2012Metric, symbol Device:C_Small
- removed C42, C43: 0.1uF, Capacitor_SMD:C_0805_2012Metric, symbol Device:C_Small
- removed C44: 0.22u, Capacitor_SMD:C_0805_2012Metric, symbol Device:C_Small
- removed C45: 10n, Capacitor_SMD:C_0805_2012Metric, symbol Device:C_Small
- removed C46: 1uF, Capacitor_SMD:C_0805_2012Metric, symbol Device:C_Small
- removed C49: 4.7u, Capacitor_SMD:C_0805_2012Metric, symbol Device:C_Small
- removed C50: 2.2u, Capacitor_SMD:C_0805_2012Metric, symbol Device:C_Small
- removed C51, C52, C53, C54, C55, C56, C57, C58: 0.1u, Capacitor_SMD:C_0805_2012Metric, symbol Device:C
- removed D1: LED, LED_SMD:LED_0805_2012Metric, symbol Device:LED
- removed J1: TEST, Connector_PinHeader_2.54mm:PinHeader_1x02_P2.54mm_Vertical, symbol Connector_Generic:Conn_01x02
- removed J10: NTC-5, Connector_PinHeader_2.54mm:PinHeader_1x02_P2.54mm_Vertical, symbol Connector_Generic:Conn_01x02
- removed J11: NTC-6, Connector_PinHeader_2.54mm:PinHeader_1x02_P2.54mm_Vertical, symbol Connector_Generic:Conn_01x02
- removed J12: NTC-7, Connector_PinHeader_2.54mm:PinHeader_1x02_P2.54mm_Vertical, symbol Connector_Generic:Conn_01x02
- removed J13: NTC-8, Connector_PinHeader_2.54mm:PinHeader_1x02_P2.54mm_Vertical, symbol Connector_Generic:Conn_01x02
- removed J2: LOW SIDE, Footprints:705510038, symbol 705510038:705510038
- removed J3: 12S, Connector_PinHeader_2.54mm:PinHeader_1x02_P2.54mm_Vertical, symbol Connector_Generic:Conn_01x02
- removed J5: HIGH SIDE, Footprints:705510038, symbol 705510038:705510038
- removed J6: NTC-1, Connector_PinHeader_2.54mm:PinHeader_1x02_P2.54mm_Vertical, symbol Connector_Generic:Conn_01x02
- removed J7: NTC-2, Connector_PinHeader_2.54mm:PinHeader_1x02_P2.54mm_Vertical, symbol Connector_Generic:Conn_01x02
- removed J8: NTC-3, Connector_PinHeader_2.54mm:PinHeader_1x02_P2.54mm_Vertical, symbol Connector_Generic:Conn_01x02
- removed J9: NTC-4, Connector_PinHeader_2.54mm:PinHeader_1x02_P2.54mm_Vertical, symbol Connector_Generic:Conn_01x02
- removed R1, R2, R23, R24, R25, R26, R27, R28, R29, R3, R30, R4, R5, R6, R7, R8, R9: 10, Resistor_SMD:R_1210_3225Metric, symbol Device:R_US
- removed R10, R11, R21, R22, R48, R49, R53, R54: 0, Resistor_SMD:R_0805_2012Metric, symbol Device:R_US
- removed R12, R13, R14, R15, R16, R17, R18, R19, R20, R33, R34, R35, R36, R37, R38, R39, R40: 100, Resistor_SMD:R_0805_2012Metric, symbol Device:R_US
- removed R31, R32, R45, R46: 51, Resistor_SMD:R_0805_2012Metric, symbol Device:R_US
- removed R41, R42, R43, R44: 499, Resistor_SMD:R_0805_2012Metric, symbol Device:R_US
- removed R47: 30, Resistor_SMD:R_2010_5025Metric, symbol Device:R_US
- removed R50: 100, Resistor_SMD:R_2010_5025Metric, symbol Device:R_US
- removed R51: 200, Resistor_SMD:R_2010_5025Metric, symbol Device:R_US
- removed R52: 4.7k, Resistor_SMD:R_2010_5025Metric, symbol Device:R_US
- removed R55, R56, R57, R58, R59, R60, R61, R62: 10.0k, Resistor_SMD:R_0805_2012Metric, symbol Device:R_US
- removed T1, T2: CEP99-102, Footprints:CEP99102, symbol CEP99-102:CEP99-102
- removed TP1, TP10, TP11, TP12, TP13, TP14, TP15, TP16, TP17, TP18, TP19, TP2, TP20, TP21, TP22, TP23, TP24, TP25, TP26, TP27, TP3, TP4, TP5, TP6, TP7, TP8, TP9: TestPoint_Square, TestPoint:TestPoint_THTPad_D1.5mm_Drill0.7mm, symbol Connector:TestPoint_Square
- removed U1, U2: PESD5V0L2BT, Footprints:SOT23_NEX, symbol PESD5V0L2BT:PESD5V0L2BT
- removed U3: ZXTN4004KQTC, Footprints:DPAK_04KQTC_DIO, symbol ZXTN4004KQTC:ZXTN4004KQTC
- removed U4: PBQ79616PAPTQ1, Footprints:PAP0064F-IPC_A, symbol BQ79616PAPRQ1:BQ79616PAPRQ1
- added F1, F10, F11, F12, F13, F14, F15, F16, F17, F18, F2, F3, F4, F5, F6, F7, F8, F9: 1A, Fuse:Fuse_0805_2012Metric, symbol Device:Fuse_Small
- added J14: JUMPER, Connector_PinHeader_2.54mm:PinHeader_2x16_P2.54mm_Vertical, symbol Connector_Generic:Conn_02x16_Counter_Clockwise
- added J2: LOW SIDE, Footprints:705510038, symbol Connector_Generic:Conn_01x04
- added J5: HIGH SIDE, Footprints:705510038, symbol Connector_Generic:Conn_01x04
- J4: symbol 705550056:705550056 -> Connector_Generic:Conn_01x22
Connections:
- net CELL0: no longer J4.21
- net CELL10: now also F11.2
- net CELL11: now also F12.2
- net CELL12: now also F13.2
- net CELL13: now also F14.2
- net CELL14: now also F15.2
- net CELL15: now also F16.2
- net CELL16S: now also F17.2
- net CELL4: now also F5.2
- net CELL5: now also F6.2
- net CELL6: now also F7.2
- net CELL7: now also F8.2
- net CELL8: now also F9.2
- net CELL9: now also F10.2
- net CELL1 renamed CELL1-UNP
- net CELL1-UNP: now also F2.2
- net CELL16 renamed CELL16-UNP
- net CELL16-UNP: now also J4.21 (Pin_21), F1.2, F18.2
- net CELL2 renamed CELL2-UNP
- net CELL2-UNP: now also F3.2
- net CELL3 renamed CELL3-UNP
- net CELL3-UNP: now also F4.2
- new net: F1.1, F18.1, J14.16 (Pin_16)
- new net BQ79616/PWR: J14.17 (Pin_17), J14.18 (Pin_18), J14.19 (Pin_19), J14.20 (Pin_20), J14.21 (Pin_21), J14.22 (Pin_22), J14.23 (Pin_23), J14.24 (Pin_24), J14.25 (Pin_25), J14.26 (Pin_26), J14.27 (Pin_27), J14.28 (Pin_28), J14.29 (Pin_29), J14.30 (Pin_30), J14.31 (Pin_31), J14.32 (Pin_32)
- new net Cell filtering and balancing/CELL1: F2.1, J14.1 (Pin_1)
- new net Cell filtering and balancing/CELL10: F11.1, J14.10 (Pin_10)
- new net Cell filtering and balancing/CELL11: F12.1, J14.11 (Pin_11)
- new net Cell filtering and balancing/CELL12: F13.1, J14.12 (Pin_12)
- new net Cell filtering and balancing/CELL13: F14.1, J14.13 (Pin_13)
- new net Cell filtering and balancing/CELL14: F15.1, J14.14 (Pin_14)
- new net Cell filtering and balancing/CELL15: F16.1, J14.15 (Pin_15)
- new net Cell filtering and balancing/CELL16S: F17.1
- new net Cell filtering and balancing/CELL2: F3.1, J14.2 (Pin_2)
- new net Cell filtering and balancing/CELL3: F4.1, J14.3 (Pin_3)
- new net Cell filtering and balancing/CELL4: F5.1, J14.4 (Pin_4)
- new net Cell filtering and balancing/CELL5: F6.1, J14.5 (Pin_5)
- new net Cell filtering and balancing/CELL6: F7.1, J14.6 (Pin_6)
- new net Cell filtering and balancing/CELL7: F8.1, J14.7 (Pin_7)
- new net Cell filtering and balancing/CELL8: F9.1, J14.8 (Pin_8)
- new net Cell filtering and balancing/CELL9: F10.1, J14.9 (Pin_9)
- new net Transformer Isolation/ISO_COMHN: J5.4 (Pin_4)
- new net Transformer Isolation/ISO_COMHP: J5.3 (Pin_3)
- new net Transformer Isolation/ISO_COMLN: J2.1 (Pin_1)
- new net Transformer Isolation/ISO_COMLP: J2.2 (Pin_2)
- no-connect marks 7 -> 4
Other:
- added sheet BQ79616 (cmu-BQ79616.kicad_sch)
- added sheet Cell filtering and balancing (cmu-cell-filtering.kicad_sch)
- added sheet Transformer Isolation (cmu-isolation.kicad_sch)
- note added: "Jumper block for power choice (Top of stack powers IC)"
- note removed: "16S default: connect CELL0-CELL16 normally. 12S test: short CELL13-CELL16 and PWR/BAT to CELL12. Do not leave unused upper channels floating."
- note removed: "BAT_TOP provides the stack-powered input for the BQ79616."
- note removed: "BQ79616 External NPN Power Path"
- note removed: "CELL0 is the local cell-stack reference for the CMU, not chassis ground."
- note removed: "Cell connector follows the TI EVM-style sensing structure. CELL0/CELL16 are stack endpoints; CELL0S/CELL16S are sense lines."
- note removed: "GPIO1-GPIO6: NTC inputs for 12S test. GPIO7-GPIO8: reserved for 16S build."
- note removed: "GPIO1–GPIO8 are routed to NTC headers for external temperature sensing."
- note removed: "GPIOs Temperature Sensing"
- note removed: "Middle module: use both COMH and COML. End module: use one side and terminate the unused side. Ring: use both sides and terminate chain ends."
- note removed: "TSREF provides the NTC bias reference."
- note removed: "Tranformer Isolation For COM Communication"
- note removed: "VB / CB"
- note removed: "VC inputs use 100Ω series resistors and 0.47uF capacitors to CELL0 for filtering."

Commit message: updated cmu layout
Parts:
- renumbered F18 to F17, F17 to F18, J4 to J1, J14 to J2, J5 to J3, J2 to J4
Other:
- sheet BQ79616 renamed CMU-BQ79616 AFE Core
- sheet Cell filtering and balancing renamed CMU-Cell Filtering & Balancing
- sheet Transformer Isolation renamed CMU-Daisy-Chain Interface
- note added: "16 CELLS"
- note removed: "CELLS"
- moved on the sheet: F1, F10, F11, F12, F13, F14, F15, F16, F17, F18, F2, F3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

Commit message: change iso+update cmu BOM
Parts:
- F1, F10, F11, F12, F13, F14, F15, F16, F17, F18, F2, F3, F4, F5, F6, F7, F8, F9: DIS (none) -> DigiKey; DPN (none) -> 478-F0805B1R00FSCT-ND; MFR (none) -> KYOCERA AVX; MPN (none) -> F0805B1R00FSTR; Purchase Link (none) -> https://www.digikey.com/en/products/detail/kyocera-avx/F080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
- J1: DIS (none) -> Mouser; DPN (none) -> 538-70555-0056; MFR (none) -> Molex; MPN (none) -> 70555-0056; Purchase Link (none) -> https://www.mouser.com/ProductDetail/Molex/70555-0056?qs=RQ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
- J3, J4: DIS (none) -> DigiKey; DPN (none) -> WM14059-ND; MFR (none) -> Molex; MPN (none) -> 705510038; Purchase Link (none) -> https://www.digikey.com/en/products/detail/molex/0705510038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

Commit message: add jumper+ change SW for bmu
Parts:
- J2: DIS (none) -> DigiKey; DPN (none) -> SAM1028-16-ND; MFR (none) -> Samtec Inc.; MPN (none) -> TSW-116-07-G-D; Purchase Link (none) -> https://www.digikey.com/en/products/detail/samtec-inc/TSW-1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; now fitted
Changed lines of the file:
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@@
 		(on_board yes)
 		(in_pos_files yes)
-		(dnp yes)
+		(dnp no)
 		(property "Reference" "J2"
 			(at 135.89 95.25 0)
@@
 			(at 156.21 96.52 0)
 			(hide yes)
+			(show_name no)
+			(do_not_autoplace no)
+			(effects
+				(font
+					(size 1.27 1.27)
+				)
+			)
+		)
+		(property "DIS" "DigiKey"
+			(at 156.21 96.52 0)
+			(hide yes)
+			(show_name no)
+			(do_not_autoplace no)
+			(effects
+				(font
+					(size 1.27 1.27)
+				)
+			)
+		)
+		(property "DPN" "SAM1028-16-ND"
+			(at 156.21 96.52 0)
+			(hide yes)
+			(show_name no)
+			(do_not_autoplace no)
+			(effects
+				(font
+					(size 1.27 1.27)
+				)
+			)
+		)
+		(property "MFR" "Samtec Inc."
+			(at 156.21 96.52 0)
+			(hide yes)
+			(show_name no)
+			(do_not_autoplace no)
+			(effects
+				(font
+					(size 1.27 1.27)
+				)
+			)
+		)
+		(property "MPN" "TSW-116-07-G-D"
+			(at 156.21 96.52 0)
+			(hide yes)
+			(show_name no)
+			(do_not_autoplace no)
+			(effects
+				(font
+					(size 1.27 1.27)
+				)
+			)
+		)
+		(property "Purchase Link" "https://www.digikey.com/en/products/detail/samtec-inc/TSW-116-07-T-D/1101561?utm_source=chatgpt.com&oppcref=6cdbc333-f2d1-4e89-ac93-8aaded010a39"
+			(at 156.21 96.52 0)
+			(hide yes)
