File: Hardware/Cell Monitoring Unit (CMU)/cmu-BQ79616.kicad_sch (KiCad schematic)
At the start: 49 parts, among them J10 NTC-5, J11 NTC-6, J12 NTC-7, J13 NTC-8, J6 NTC-1, J7 NTC-2, J8 NTC-3, J9 NTC-4, U3 ZXTN4004KQTC, U4 PBQ79616PAPTQ1

Commit message: A bit more schematic polishing
Parts:
- removed C49: 4.7u, Capacitor_SMD:C_0805_2012Metric, symbol Device:C_Small
- added C59: 4.7u, Capacitor_SMD:C_0805_2012Metric, symbol Device:C_Small
- D1: value LED -> GRN
Connections:
- net CELL0: now also C59.2
- net at R52.1, TP20.1, U4.45 (CVDD)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: now also C59.1
Other:
- note added: "Leave floating if not bottom battery pack; probably just don't use"
- note added: "Not used; pull to CVDD"
- note added: "Power LED"
- note removed: "16S default: connect CELL0-CELL16 normally. 12S test: short CELL13-CELL16 and PWR/BAT to CELL12. Do not leave unused upper channels floating."
- note removed: "GPIO1-GPIO6: NTC inputs for 12S test. GPIO7-GPIO8: reserved for 16S build."
- note removed: "Middle module: use both COMH and COML. End module: use one side and terminate the unused side. Ring: use both sides and terminate chain ends."
- moved on the sheet: C41, C42, D1, J10, J11, J12, J13, J6, J7, J8, J9, R52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

Commit message: updated cmu layout
Parts:
- removed C59: 4.7u, Capacitor_SMD:C_0805_2012Metric, symbol Device:C_Small
- added C40: 4.7u, Capacitor_SMD:C_0805_2012Metric, symbol Device:C_Small
- renumbered C43 to C35, C44 to C36, C45 to C37, C46 to C38, C48 to C39, C42 to C41, C50 to C42, C41 to C43, C51 to C44, C52 to C45, C53 to C46, C54 to C47, C55 to C48, C56 to C49, C57 to C50, C58 to C51, J11 to J10, J12 to J11, J13 to J12, J6 to J5, J7 to J6, J8 to J7, J9 to J8, J10 to J9, R50 to R35, R51 to R36, R47 to R37, R52 to R38, R55 to R39, R56 to R40, R57 to R41, R58 to R42, R59 to R43, R60 to R44, R61 to R45, R62 to R46, TP19 to TP18, TP20 to TP19, TP21 to TP20, TP23 to TP21, TP24 to TP22, TP25 to TP23, TP26 to TP24, TP27 to TP25, TP22 to TP26, U3 to U1, U4 to U2
Connections:
- net CELL0: now also C40.2
- net at R38.1, TP19.1, U2.45 (CVDD)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: now also C40.1
Other:
- note added: "PWR provides the stack-powered input for the BQ79616."
- note removed: "BAT_TOP provides the stack-powered input for the BQ79616."
- moved on the sheet: C35, C36, C37, C38, C39, C41, C42, C43, C44, C45, C46, C47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

Commit message: change iso+update cmu BOM
Parts:
- C35, C41, C44, C45, C46, C47, C48, C49, C50, C51: DIS (none) -> DigiKey; DPN (none) -> 4587-C0805X104K050TCT-ND; MFR (none) -> Holy Stone Enterprise; MPN (none) -> C0805X104K050T; Purchase Link (none) -> https://www.digikey.com/en/products/detail/holy-stone-enter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
- C36: DIS (none) -> DigiKey; DPN (none) -> 732-13196-1-ND; MFR (none) -> Würth Elektronik; MPN (none) -> 8.85382E+11; Purchase Link (none) -> https://www.digikey.com/en/products/detail/w%C3%BCrth-elekt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
- C37: DIS (none) -> DigiKey; DPN (none) -> 399-17885-1-ND; MFR (none) -> KEMET; MPN (none) -> C0805C103K5RECAUTO; Purchase Link (none) -> https://www.digikey.com/en/products/detail/kemet/C0805C103K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
- C38, C39, C43: DIS (none) -> DigiKey; DPN (none) -> 399-C0805C105K5RACTUCT-ND; MFR (none) -> KEMET; MPN (none) -> C0805C105K5RACTU; Purchase Link (none) -> https://www.digikey.com/en/products/detail/kemet/C0805C105K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
- C40: DIS (none) -> DigiKey; DPN (none) -> 4587-C0805X475K025TCT-ND; MFR (none) -> Holy Stone Enterprise; MPN (none) -> C0805X475K025T; Purchase Link (none) -> https://www.digikey.com/en/products/detail/holy-stone-enter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
- C42: DIS (none) -> DigiKey; DPN (none) -> 732-7673-1-ND; MFR (none) -> Würth Elektronik; MPN (none) -> 8.85012E+11; Purchase Link (none) -> https://www.digikey.com/en/products/detail/w%C3%BCrth-elekt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
- D1: DIS (none) -> DigiKey; DPN (none) -> 160-1414-1-ND; MFR (none) -> Lite-On; MPN (none) -> LTST-C170KGKT; Purchase Link (none) -> https://www.digikey.com/en/products/detail/liteon/LTST-C170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
- J10, J11, J12, J5, J6, J7, J8, J9: DIS (none) -> DigiKey; DPN (none) -> 732-5315-ND; MFR (none) -> Würth Elektronik; MPN (none) -> 61300211121; Purchase Link (none) -> https://www.digikey.com/en/products/detail/w%C3%BCrth-elekt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
- R35: DIS (none) -> DigiKey; DPN (none) -> RMCF2010FT100RCT-ND; MFR (none) -> Stackpole Electronics; MPN (none) -> RMCF2010FT100R; Purchase Link (none) -> https://www.digikey.com/en/products/detail/stackpole-electr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
- R36: DIS (none) -> DigiKey; DPN (none) -> RMCF2010FT200RCT-ND; MFR (none) -> Stackpole Electronics; MPN (none) -> RMCF2010FT200R; Purchase Link (none) -> https://www.digikey.com/en/products/detail/stackpole-electr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
- R37: DIS (none) -> DigiKey; DPN (none) -> 13-RC2010FK-0730RLCT-ND; MFR (none) -> YAGEO; MPN (none) -> RC2010FK-0730RL; Purchase Link (none) -> https://www.digikey.com/en/products/detail/yageo/RC2010FK-0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
- R38: DIS (none) -> DigiKey; DPN (none) -> 13-RC2010FK-074K7LCT-ND; MFR (none) -> YAGEO; MPN (none) -> RC2010FK-074K7L; Purchase Link (none) -> https://www.digikey.com/en/products/detail/yageo/RC2010FK-0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
- R39, R40, R41, R42, R43, R44, R45, R46: DIS (none) -> DigiKey; DPN (none) -> 311-10.0KCRCT-ND; MFR (none) -> YAGEO; MPN (none) -> RC0805FR-0710KL; Purchase Link (none) -> https://www.digikey.com/en/products/detail/yageo/RC0805FR-0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
- U1: DIS (none) -> DigiKey; DPN (none) -> 31-ZXTN4004KQTCCT-ND; MFR (none) -> Diodes Incorporated; MPN (none) -> ZXTN4004KQTC; Purchase Link (none) -> https://www.digikey.com/en/products/detail/diodes-incorpora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
- U2: DIS (none) -> DigiKey; DPN (none) -> 296-BQ79616PAPRQ1CT-ND; MFR (none) -> Texas Instruments; MPN (none) -> BQ79616PAPRQ1; Purchase Link (none) -> https://www.digikey.com/en/products/detail/texas-instrument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

Commit message: finish! update bmu layout+BOM
Parts:
- C36: MPN 8.85382E+11 -> 885382207008
- C38: value 1uF -> 1u
- C42: MPN 8.85012E+11 -> 885012207079
Changed lines of the file:
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@@
 			)
 		)
-		(property "Value" "1uF"
+		(property "Value" "1u"
 			(at 144.78 156.2165 0)
 			(show_name no)
@@
 			)
 		)
-		(property "MPN" "8.85382E+11"
+		(property "MPN" "885382207008"
 			(at 86.36 137.16 0)
 			(hide yes)
@@
 			)
 		)
-		(property "MPN" "8.85012E+11"
+		(property "MPN" "885012207079"
 			(at 170.18 153.67 0)
 			(hide yes)
