File: Hardware/Cell Monitoring Unit (CMU)/cmu-cell-filtering.kicad_sch (KiCad schematic)
At the start: 85 parts

Commit message: updated cmu layout
Parts:
- renumbered C21 to C19, C22 to C20, C23 to C21, C24 to C22, C25 to C23, C26 to C24, C27 to C25, C28 to C26, C30 to C27, C31 to C28, C32 to C29, C33 to C30, C34 to C31, C35 to C32, C36 to C33, C37 to C34, R12 to R10, R13 to R11, R14 to R12, R15 to R13, R16 to R14, R17 to R15, R18 to R16, R19 to R17, R20 to R18, R23 to R19, R24 to R20, R25 to R21, R26 to R22, R27 to R23, R28 to R24, R29 to R25, R30 to R26, R33 to R27, R34 to R28, R35 to R29, R36 to R30, R37 to R31, R38 to R32, R39 to R33, R40 to R34, TP11 to TP10, TP12 to TP11, TP13 to TP12, TP14 to TP13, TP15 to TP14, TP16 to TP15, TP17 to TP16, TP18 to TP17
Other:
- moved on the sheet: C1, C10, C11, C12, C13, C14, C15, C16, C17, C18, C19, C2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

Commit message: change iso+update cmu BOM
Parts:
- C1, C10, C11, C12, C13, C14, C15, C16, C17, C18, C19, C2, C20, C21, C22, C23, C24, C25, C26, C27, C28, C29, C3, C30, C31, C32, C33, C34, C4, C5, C6, C7, C8, C9: DIS (none) -> DigiKey; DPN (none) -> 13-CS0805KKX7R9BB474CT-ND; MFR (none) -> YAGEO; MPN (none) -> CS0805KKX7R9BB474; Purchase Link (none) -> https://www.digikey.com/en/products/detail/yageo/CS0805KKX7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
- R1, R19, R2, R20, R21, R22, R23, R24, R25, R26, R3, R4, R5, R6, R7, R8, R9: DIS (none) -> DigiKey; DPN (none) -> 13-RC1210FR-0710RLCT-ND; MFR (none) -> YAGEO; MPN (none) -> RC1210FR-0710RL; Purchase Link (none) -> https://www.digikey.com/en/products/detail/yageo/RC1210FR-0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
- R10, R11, R12, R13, R14, R15, R16, R17, R18, R27, R28, R29, R30, R31, R32, R33, R34: DIS (none) -> DigiKey; DPN (none) -> 311-100CRCT-ND; MFR (none) -> YAGEO; MPN (none) -> RC0805FR-07100RL; Purchase Link (none) -> https://www.digikey.com/en/products/detail/yageo/RC0805FR-0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
